Commit message: first attempt at gazebo, able to launch in empty world but there are still many bugs

File: src/mir_description/urdf/include/imu.gazebo.urdf.xacro (robot description, xacro)
@@ -1,27 +1,28 @@
 <?xml version="1.0"?>
 <robot xmlns:xacro="http://ros.org/wiki/xacro">
-  <!-- If tf_prefix is given, use "frame tf_prefix/imu_frame", else "imu_frame" -->
   <xacro:arg name="tf_prefix" default="" />
-  <xacro:property name="tf_prefix" value="$(arg tf_prefix)" />
-  <xacro:if value="${tf_prefix == ''}">
-      <xacro:property name="imu_frame" value="imu_frame" />
-  </xacro:if>
-  <xacro:unless value="${tf_prefix == ''}">
-      <xacro:property name="imu_frame" value="$(arg tf_prefix)/imu_frame" />
-  </xacro:unless>
+  <xacro:property name="prefix" value="$(arg tf_prefix)" />
+  <xacro:property name="imu_frame" value="${prefix + '/imu_frame' if prefix != '' else 'imu_frame'}" />
   <xacro:macro name="imu_gazebo" params="link imu_topic update_rate">
-    <gazebo>
-      <plugin name="imu_plugin" filename="libhector_gazebo_ros_imu.so">
-        <updateRate>${update_rate}</updateRate>
-        <bodyName>${link}</bodyName>
-        <frameId>${imu_frame}</frameId>  <!-- from real MiR -->
-        <topicName>${imu_topic}</topicName>
-        <accelDrift>0.0 0.0 0.0</accelDrift>
-        <accelGaussianNoise>${sqrt(5e-05)} ${sqrt(0.0001)} ${sqrt(0.00013)}</accelGaussianNoise>    <!-- real MiR linear_acceleration_covariance: [5e-05, 0.0, 0.0, 0.0, 0.0001, 0.0, 0.0, 0.0, 0.00013] -->
-        <rateDrift>0.0 0.0 0.0</rateDrift>
-        <rateGaussianNoise>${sqrt(8e-06)} ${sqrt(8e-06)} ${sqrt(3e-07)}</rateGaussianNoise>         <!-- real MiR angular_velocity_covariance: [8e-06, 0.0, 0.0, 0.0, 8e-06, 0.0, 0.0, 0.0, 3e-07] -->
-        <yawDrift>0.0</yawDrift>
-        <yawGaussianNoise>${sqrt(0.1)}</yawGaussianNoise>                                           <!-- real MiR orientation_covariance: [0.1, 0.0, 0.0, 0.0, 0.1, 0.0, 0.0, 0.0, 0.1] -->
-      </plugin>
+    <gazebo reference="${link}">
+      <sensor name="${link}_imu" type="imu">
+        <always_on>true</always_on>
+        <update_rate>${update_rate}</update_rate>
+        <visualize>false</visualize>
+        <topic>${imu_topic}</topic>
+        <gz_frame_id>${imu_frame}</gz_frame_id>
+        <imu>
+          <angular_velocity>
+            <x><noise type="gaussian"><mean>0.0</mean><stddev>${sqrt(8e-06)}</stddev></noise></x>
+            <y><noise type="gaussian"><mean>0.0</mean><stddev>${sqrt(8e-06)}</stddev></noise></y>
+            <z><noise type="gaussian"><mean>0.0</mean><stddev>${sqrt(3e-07)}</stddev></noise></z>
+          </angular_velocity>
+          <linear_acceleration>
+            <x><noise type="gaussian"><mean>0.0</mean><stddev>${sqrt(5e-05)}</stddev></noise></x>
+            <y><noise type="gaussian"><mean>0.0</mean><stddev>${sqrt(0.0001)}</stddev></noise></y>
+            <z><noise type="gaussian"><mean>0.0</mean><stddev>${sqrt(0.00013)}</stddev></noise></z>
+          </linear_acceleration>
+        </imu>
+      </sensor>
     </gazebo>
   </xacro:macro>

File: src/mir_description/urdf/include/mir_v1.urdf.xacro (robot description, xacro)
@@ -1,15 +1,10 @@
 <?xml version="1.0"?>
 <robot xmlns:xacro="http://ros.org/wiki/xacro">
-  <xacro:arg name="mir_type" default="mir_100" />      <!-- The MiR variant. Can be "mir_100" or "mir_250" for now.-->
-  <xacro:property name="mir_type" value="$(arg mir_type)" />  <!-- necessary because args cannot be accessed inside ${} expressions -->
+  <xacro:arg name="mir_type" default="mir_100" />
+  <xacro:property name="mir_type" value="$(arg mir_type)" />
   <xacro:include filename="$(find mir_description)/urdf/include/common_properties.urdf.xacro" />
   <xacro:include filename="$(find mir_description)/urdf/include/imu.gazebo.urdf.xacro" />
-  <xacro:include filename="$(find mir_description)/urdf/include/mir.gazebo.xacro" />
-  <xacro:include filename="$(find mir_description)/urdf/include/mir.transmission.xacro" />
   <xacro:include filename="$(find mir_description)/urdf/include/sick_s300.urdf.xacro" />
   <xacro:property name="deg_to_rad" value="0.017453293" />
-  <!-- The inertia for the MiR platform is intentionally chosen to be smaller than
-       the bounding box and also shifted a bit to the back, because most of the mass
-       is in the lower center back (because of the batteries). -->
   <xacro:property name="mir_base_inertial_x" value="-0.05" />
   <xacro:property name="mir_base_inertial_y" value="0.0" />
@@ -25,12 +20,8 @@
     <xacro:property name="mir_act_wheel_dx" value="0.037646" />
     <xacro:property name="mir_act_wheel_dy" value="0.222604" />
-  </xacro:if>
-  <xacro:if value="${mir_type == 'mir_250'}">
-    <xacro:property name="mir_base_mass" value="97.0" />
-    <xacro:property name="mir_act_wheel_radius" value="0.100" />
-    <xacro:property name="mir_act_wheel_width" value="0.038" />
-    <xacro:property name="mir_act_wheel_mass" value="1.0" />
-    <xacro:property name="mir_act_wheel_dx" value="-0.004485" />
-    <xacro:property name="mir_act_wheel_dy" value="0.2015" />
+    <xacro:property name="mir_back_caster_wheel_base_dx"  value="0.3078" />
+    <xacro:property name="mir_caster_wheel_base_dy" value="0.203" />
+    <xacro:property name="laser_dx" value="0.392" />
+    <xacro:property name="laser_dy" value="0.2358" />
   </xacro:if>
   <xacro:property name="mir_caster_wheel_radius" value="0.0625" />
@@ -41,22 +32,5 @@
   <xacro:property name="mir_caster_wheel_dz" value="-0.094" />
   <xacro:property name="mir_front_caster_wheel_base_dx" value="0.3037" />
-  <xacro:if value="${mir_type == 'mir_100'}">
-    <xacro:property name="mir_back_caster_wheel_base_dx"  value="0.3078" />
-    <xacro:property name="mir_caster_wheel_base_dy" value="0.203" />
-  </xacro:if>
-  <xacro:if value="${mir_type == 'mir_250'}">
-    <xacro:property name="mir_back_caster_wheel_base_dx"  value="0.296" />
-    <xacro:property name="mir_caster_wheel_base_dy" value="0.188" />
-  </xacro:if>
   <xacro:property name="mir_caster_wheel_base_dz" value="${mir_caster_wheel_radius - mir_caster_wheel_dz}" />
-  <!-- from visually matching up the meshes of the MiR and the laser scanner -->
-  <xacro:if value="${mir_type == 'mir_100'}">
-    <xacro:property name="laser_dx" value="0.392" />
-    <xacro:property name="laser_dy" value="0.2358" />
-  </xacro:if>
-  <xacro:if value="${mir_type == 'mir_250'}">
-    <xacro:property name="laser_dx" value="0.315" />
-    <xacro:property name="laser_dy" value="0.205" />
-  </xacro:if>
   <xacro:property name="laser_dz" value="0.1914" />
   <xacro:macro name="actuated_wheel" params="prefix locationprefix locationright">
@@ -74,22 +48,35 @@
       <visual>
         <origin xyz="0 0 0" rpy="${pi/2} 0 0" />
-        <geometry>
-          <cylinder radius="${mir_act_wheel_radius}" length="${mir_act_wheel_width}" />
-        </geometry>
+        <geometry><cylinder radius="${mir_act_wheel_radius}" length="${mir_act_wheel_width}" /></geometry>
         <xacro:insert_block name="material_black" />
       </visual>
       <collision>
         <origin xyz="0 0 0" rpy="${pi/2} 0 0" />
-        <geometry>
-          <cylinder radius="${mir_act_wheel_radius}" length="${mir_act_wheel_width}" />
-        </geometry>
+        <geometry><cylinder radius="${mir_act_wheel_radius}" length="${mir_act_wheel_width}" /></geometry>
       </collision>
     </link>
     <gazebo reference="${prefix}${locationprefix}_wheel_link">
-      <material>Gazebo/FlatBlack</material>
+      <visual>
+        <material>
+          <ambient>0.1 0.1 0.1 1</ambient>
+          <diffuse>0.1 0.1 0.1 1</diffuse>
+        </material>
+      </visual>
+      <collision>
+        <surface>
+          <friction>
+            <ode>
+              <mu>1.0</mu>
+              <mu2>1.0</mu2>
+              <fdir1>0 0 0</fdir1>
+              <slip1>0.0</slip1>
+              <slip2>0.0</slip2>
+            </ode>
+          </friction>
+        </surface>
+      </collision>
     </gazebo>
   </xacro:macro>
   <xacro:macro name="caster_wheel" params="prefix locationprefix locationright wheel_base_dx">
-    <!-- caster hub -->
     <joint name="${prefix}${locationprefix}_caster_rotation_joint" type="continuous">
       <origin xyz="${wheel_base_dx} ${-mir_caster_wheel_base_dy * locationright} ${mir_caster_wheel_base_dz}" rpy="0 0 0" />
@@ -101,14 +88,7 @@
     <link name="${prefix}${locationprefix}_caster_rotation_link">
       <inertial>
-        <!-- <origin xyz="0 0 -0.042500000044" rpy="${0.5 * pi} ${24 * deg_to_rad} ${1.5 * pi}" /> -->
         <origin xyz="0 0 -0.042500000044" rpy="${24 * deg_to_rad} 0 ${0.5 * pi} " />
         <mass value="0.3097539019" />
-        <inertia
-          ixx="0.0005844517978"
-          ixy="0"
-          ixz="0"
-          iyy="0.00052872551237"
-          iyz="0"
-          izz="0.00017923555074" />
+        <inertia ixx="0.0005844517978" ixy="0" ixz="0" iyy="0.00052872551237" iyz="0" izz="0.00017923555074" />
       </inertial>
       <visual>
@@ -117,10 +97,5 @@
           <mesh filename="package://mir_description/meshes/visual/caster_wheel_base.stl" />
         </geometry>
-        <xacro:if value="${mir_type == 'mir_100'}">
-          <xacro:insert_block name="material_silver" />
-        </xacro:if>
-        <xacro:if value="${mir_type == 'mir_250'}">
-          <xacro:insert_block name="material_black" />
-        </xacro:if>
+        <xacro:insert_block name="material_silver" />
       </visual>
       <collision>
@@ -131,13 +106,4 @@
       </collision>
     </link>
-    <gazebo reference="${prefix}${locationprefix}_caster_rotation_link">
-      <xacro:if value="${mir_type == 'mir_100'}">
-        <material>Gazebo/Grey</material>
-      </xacro:if>
-      <xacro:if value="${mir_type == 'mir_250'}">
-        <material>Gazebo/FlatBlack</material>
-      </xacro:if>
-    </gazebo>
-    <!-- caster wheel -->
     <joint name="${prefix}${locationprefix}_caster_wheel_joint" type="continuous">
       <origin xyz="${mir_caster_wheel_dx} ${-mir_caster_wheel_dy * locationright} ${mir_caster_wheel_dz}" rpy="0 0 0" />
@@ -152,18 +118,30 @@
       <visual>
         <origin xyz="0 0 0" rpy="${pi/2} 0 0" />
-        <geometry>
-          <cylinder radius="${mir_caster_wheel_radius}" length="${mir_caster_wheel_width}" />
-        </geometry>
+        <geometry><cylinder radius="${mir_caster_wheel_radius}" length="${mir_caster_wheel_width}" /></geometry>
         <xacro:insert_block name="material_black" />
       </visual>
       <collision>
         <origin xyz="0 0 0" rpy="${pi/2} 0 0" />
-        <geometry>
-          <cylinder radius="${mir_caster_wheel_radius}" length="${mir_caster_wheel_width}" />
-        </geometry>
+        <geometry><cylinder radius="${mir_caster_wheel_radius}" length="${mir_caster_wheel_width}" /></geometry>
       </collision>
     </link>
     <gazebo reference="${prefix}${locationprefix}_caster_wheel_link">
-      <material>Gazebo/FlatBlack</material>
+      <visual>
+        <material>
+          <ambient>0.1 0.1 0.1 1</ambient>
+          <diffuse>0.1 0.1 0.1 1</diffuse>
+        </material>
+      </visual>
+      <collision>
+        <surface>
+          <friction>
+            <ode>
+              <mu>0.0</mu> <mu2>0.0</mu2>
+              <slip1>1.0</slip1>
+              <slip2>1.0</slip2>
+            </ode>
+          </friction>
+        </surface>
+      </collision>
     </gazebo>
   </xacro:macro>
@@ -184,10 +162,5 @@
           <mesh filename="package://mir_description/meshes/visual/${mir_type}_base.stl" />
         </geometry>
-        <xacro:if value="${mir_type == 'mir_100'}">
-          <xacro:insert_block name="material_white" />
-        </xacro:if>
-        <xacro:if value="${mir_type == 'mir_250'}">
-          <xacro:insert_block name="material_dark_grey" />
-        </xacro:if>
+        <xacro:insert_block name="material_white" />
       </visual>
       <collision>
@@ -198,23 +171,11 @@
       </collision>
     </link>
-    <gazebo reference="${prefix}base_link">
-      <xacro:if value="${mir_type == 'mir_100'}">
-        <material>Gazebo/White</material>
-      </xacro:if>
-      <xacro:if value="${mir_type == 'mir_250'}">
-        <material>Gazebo/DarkGrey</material>
-      </xacro:if>
-    </gazebo>
-    <!-- IMU -->
     <joint name="${prefix}base_link_to_imu_joint" type="fixed">
       <parent link="${prefix}base_link" />
       <child link="${prefix}imu_link" />
-      <origin xyz="0.0 0.0 0.25" rpy="0 0 0" />  <!-- same as real MiR -->
+      <origin xyz="0.0 0.0 0.25" rpy="0 0 0" />
     </joint>
     <link name="${prefix}imu_link" />
     <xacro:imu_gazebo link="${prefix}imu_link" imu_topic="imu_data" update_rate="50.0" />
-    <!-- Create an alias for imu_link. This is necessary because the real MiR's
-         TF has imu_link, but the imu_data topic is published in the imu_frame
-         frame. -->
     <joint name="${prefix}imu_link_to_imu_frame_joint" type="fixed">
       <parent link="${prefix}imu_link" />
@@ -223,5 +184,4 @@
     </joint>
     <link name="${prefix}imu_frame" />
-    <!-- Laser scanners -->
     <joint name="${prefix}base_link_to_front_laser_joint" type="fixed">
       <parent link="${prefix}base_link" />
@@ -236,18 +196,4 @@
     </joint>
     <xacro:sick_s300 prefix="${prefix}" link="back_laser_link" topic="b_scan" />
-    <!-- Ultrasound sensors -->
-    <joint name="${prefix}us_1_joint" type="fixed">   <!-- right ultrasound -->
-      <parent link="${prefix}base_link" />
-      <child link="${prefix}us_1_frame" />
-      <origin xyz="0.45 -0.12 0.16 " rpy="0 0 0" />  <!-- from visually matching to the mesh of the MiR -->
-    </joint>
-    <link name="${prefix}us_1_frame" />
-    <joint name="${prefix}us_2_joint" type="fixed">   <!-- left ultrasound -->
-      <parent link="${prefix}base_link" />
-      <child link="${prefix}us_2_frame" />
-      <origin xyz="0.45 0.12 0.16 " rpy="0 0 0" />  <!-- from visually matching to the mesh of the MiR -->
-    </joint>
-    <link name="${prefix}us_2_frame" />
-    <!-- wheels -->
     <xacro:actuated_wheel prefix="${prefix}" locationprefix="left" locationright="-1"/>
     <xacro:actuated_wheel prefix="${prefix}" locationprefix="right" locationright="1"/>
@@ -256,15 +202,4 @@
     <xacro:caster_wheel prefix="${prefix}" locationprefix="bl" locationright="-1" wheel_base_dx="${-mir_back_caster_wheel_base_dx + mir_act_wheel_dx}"/>
     <xacro:caster_wheel prefix="${prefix}" locationprefix="br" locationright="1" wheel_base_dx="${-mir_back_caster_wheel_base_dx + mir_act_wheel_dx}"/>
-    <joint name="${prefix}base_link_surface_joint" type="fixed">
-      <origin xyz="${mir_act_wheel_dx} 0 0.352" rpy="0 0 0" />
-      <parent link="${prefix}base_link" />
-      <child link="${prefix}surface" />
-      <axis xyz="0 0 1" />
-    </joint>
-    <link name="${prefix}surface"/>
-    <xacro:mir_wheel_transmissions prefix="${prefix}"/>
-    <!-- set the gazebo friction parameters for the wheels -->
-    <xacro:set_all_wheel_frictions prefix="${prefix}"/>
-    <xacro:p3d_base_controller prefix="${prefix}" />
-  </xacro:macro>
+    </xacro:macro>
 </robot>

File: src/mir_description/urdf/include/sick_s300.urdf.xacro (robot description, xacro)
@@ -13,5 +13,4 @@
           <mesh filename="package://mir_description/meshes/visual/sick_lms-100.stl" />
         </geometry>
-        <!-- <xacro:insert_block name="material_yellow" /> -->
         <xacro:insert_block name="material_black" />
       </visual>
@@ -27,15 +26,21 @@
     </link>
     <gazebo reference="${prefix}${link}">
-      <!-- <material value="Gazebo/Yellow" /> -->
-      <material value="Gazebo/FlatBlack" />
-      <sensor type="ray" name="${prefix}${link}">
+      <visual>
+        <material>
+          <ambient>0.1 0.1 0.1 1.0</ambient>
+          <diffuse>0.1 0.1 0.1 1.0</diffuse>
+        </material>
+      </visual>
+      <sensor type="gpu_lidar" name="${prefix}${link}_sensor">
         <pose>0 0 0 0 0 0</pose>
         <visualize>false</visualize>
         <update_rate>12.5</update_rate>
-        <ray>
+        <topic>${topic}</topic>
+        <gz_frame_id>${prefix}${link}</gz_frame_id>
+        <lidar>
           <scan>
             <horizontal>
               <samples>541</samples>
-              <resolution>1</resolution>  <!-- has to be 1; actual resolution will be computed from number of samples + min_angle/max_angle -->
+              <resolution>1</resolution>
               <min_angle>-2.35619449615</min_angle>
               <max_angle>2.35619449615</max_angle>
@@ -49,15 +54,8 @@
           <noise>
             <type>gaussian</type>
-            <!-- Noise parameters based on published spec for S300 achieving
-                 "+-29mm" accuracy at range < 3m (~0.01 of the range) at
-                 1 sigma. -->
             <mean>0.0</mean>
             <stddev>0.01</stddev>
           </noise>
-        </ray>
-        <plugin name="gazebo_ros_${link}_controller" filename="libgazebo_ros_laser.so">
-          <frameName>${prefix}${link}</frameName>
-          <topicName>${topic}</topicName>
-        </plugin>
+        </lidar>
       </sensor>
     </gazebo>

File: src/mir_description/urdf/mir.urdf.xacro (robot description, xacro)
@@ -1,24 +1,26 @@
 <?xml version="1.0"?>
-<robot xmlns:xacro="http://ros.org/wiki/xacro"
-       name="mir" >
-  <!-- MiR base -->
+<robot xmlns:xacro="http://ros.org/wiki/xacro" name="mir">
   <xacro:include filename="$(find mir_description)/urdf/include/mir_v1.urdf.xacro" />
-  <xacro:include filename="$(find mir_description)/urdf/include/common.gazebo.xacro" />
   <xacro:arg name="tf_prefix" default="" />
-  <xacro:property name="tf_prefix_" value="$(arg tf_prefix)" />
-  <xacro:if value="${tf_prefix_ == ''}">
-    <xacro:property name="prefix" value="" />
-  </xacro:if>
-  <xacro:unless value="${tf_prefix_ == ''}">
-    <xacro:property name="prefix" value="${tf_prefix_}/" />
-  </xacro:unless>
-  <xacro:mir prefix="${prefix}" />
-  <xacro:controller_plugin_gazebo robot_namespace=""/>
-  <!-- instead of the controller_plugin_gazebo, you can use the diffdrive controller like this:
-    <xacro:diff_controller_plugin_gazebo prefix=""
-      left_wheel_joint="left_wheel_joint"
-      right_wheel_joint="right_wheel_joint"
-      wheel_separation="${2*mir_act_wheel_dy}"
-      wheel_radius="${mir_act_wheel_radius}"/>
-  -->
+  <xacro:property name="prefix" value="$(arg tf_prefix)" />
+  <xacro:property name="prefix_with_slash" value="${prefix + '/' if prefix != '' else ''}" />
+  <xacro:mir prefix="${prefix_with_slash}" />
+  <gazebo>
+    <plugin filename="gz-sim-diff-drive-system" name="gz::sim::systems::DiffDrive">
+      <left_joint>${prefix_with_slash}left_wheel_joint</left_joint>
+      <right_joint>${prefix_with_slash}right_wheel_joint</right_joint>
+      <wheel_separation>0.445208</wheel_separation>
+      <wheel_radius>0.0625</wheel_radius>
+      <odom_publish_frequency>50</odom_publish_frequency>
+      <topic>cmd_vel</topic>
+      <odom_topic>odom</odom_topic>
+      <frame_id>odom</frame_id>
+      <child_frame_id>${prefix_with_slash}base_footprint</child_frame_id>
+    </plugin>
+    <plugin filename="gz-sim-joint-state-publisher-system" name="gz::sim::systems::JointStatePublisher">
+      <topic>joint_states</topic>
+      <joint_name>${prefix_with_slash}left_wheel_joint</joint_name>
+      <joint_name>${prefix_with_slash}right_wheel_joint</joint_name>
+    </plugin>
+  </gazebo>
 </robot>
