Commit message: optimized for simulation

File: src/mir_description/urdf/include/mir_v1.urdf.xacro (robot description, xacro)
@@ -127,23 +127,20 @@
     </link>
     <gazebo reference="${prefix}${locationprefix}_caster_wheel_link">
-      <visual>
-        <material>
-          <ambient>0.1 0.1 0.1 1</ambient>
-          <diffuse>0.1 0.1 0.1 1</diffuse>
-        </material>
-      </visual>
-      <collision>
-        <surface>
-          <friction>
-            <ode>
-              <mu>0.0</mu> <mu2>0.0</mu2>
-              <slip1>1.0</slip1>
-              <slip2>1.0</slip2>
-            </ode>
-          </friction>
-        </surface>
-      </collision>
-    </gazebo>
-  </xacro:macro>
+        <!-- These must be flat under the gazebo tag for the URDF parser to see them! -->
+        <mu1>0.0</mu1>
+        <mu2>0.0</mu2>
+        <kp>10000000.0</kp>
+        <kd>1.0</kd>
+        <minDepth>0.001</minDepth>
+        <maxVel>1.0</maxVel>
+        <!-- Keep your visual settings -->
+        <visual>
+          <material>
+            <ambient>0.1 0.1 0.1 1</ambient>
+            <diffuse>0.1 0.1 0.1 1</diffuse>
+          </material>
+        </visual>
+      </gazebo>
+    </xacro:macro>
   <xacro:macro name="mir" params="prefix">
     <link name="${prefix}base_footprint" />
@@ -177,5 +174,5 @@
     </joint>
     <link name="${prefix}imu_link" />
-    <xacro:imu_gazebo link="${prefix}imu_link" imu_topic="imu_data" update_rate="50.0" />
+    <xacro:imu_gazebo link="${prefix}imu_link" imu_topic="imu" update_rate="50.0" />
     <joint name="${prefix}imu_link_to_imu_frame_joint" type="fixed">
       <parent link="${prefix}imu_link" />

File: src/mir_description/urdf/include/sick_s300.urdf.xacro (robot description, xacro)
@@ -39,5 +39,5 @@
         <pose>0.045 0 0 0 0 0</pose>
         <visualize>true</visualize>
-        <update_rate>30.0</update_rate>
+        <update_rate>10.0</update_rate>
         <self_collide>false</self_collide>
         <topic>${topic}</topic>
@@ -47,5 +47,5 @@
           <scan>
             <horizontal>
-              <samples>541</samples>
+              <samples>360</samples>
               <resolution>1</resolution>
               <min_angle>-2.35619449615</min_angle>

File: src/mir_description/urdf/mir.urdf.xacro (robot description, xacro)
@@ -17,5 +17,5 @@
       <tf_topic>/tf</tf_topic>
       <frame_id>odom</frame_id>
-      <publish_odom_tf>true</publish_odom_tf>
+      <publish_odom_tf>false</publish_odom_tf>
       <child_frame_id>${prefix_with_slash}base_footprint</child_frame_id>
     </plugin>
